Commit message: remove some collision

File: kinetic/src/four_wheel_urdf/urdf/four_wheel_urdf.urdf (robot description, URDF)
Before this commit: robot four_wheel_urdf, 9 links, 8 joints
Links:
- link driver_link: geometry visual mesh filename=package://four_wheel_urdf/meshes/driver_link.STL
- link kinect_link: geometry visual mesh filename=package://four_wheel_urdf/meshes/kinect_link.STL
- link lidar_link: geometry visual mesh filename=package://four_wheel_urdf/meshes/lidar_link.STL
- link raspberry_link: geometry visual mesh filename=package://four_wheel_urdf/meshes/raspberry_link.STL
