Commit message: add xacro support

File: kinetic/src/four_wheel_urdf/urdf/four_wheel_urdf.urdf.xacro (robot description, xacro)
@@ -1,9 +1,11 @@
 <?xml version="1.0" encoding="utf-8"?>
+<robot xmlns:xacro="http://www.ros.org/wiki/xacro" name="four_wheel_urdf">
 <!-- This URDF was automatically created by SolidWorks to URDF Exporter! Originally created by Stephen Brawner (brawner@gmail.com)
      Commit Version: 1.5.1-0-g916b5db  Build Version: 1.5.7152.31018
      For more information, please see http://wiki.ros.org/sw_urdf_exporter -->
 <!--Model constructed by yu zhuotong 2020.5.10-->
-<robot
-  name="four_wheel_urdf">
+  <xacro:property name = "wheel_mass" value = "0.5"/>
+  <xacro:property name = "lidar_mass" value = "2"/>
+  <xacro:property name = "kinect_mass" value = "0.5"/>
   <link
     name="base_link">
@@ -53,5 +55,9 @@
         rpy="0 0 0" />
       <mass
+        value="${wheel_mass}" />
+      <!--
+      <mass
         value="0.186539970489831" />
+      -->
       <inertia
         ixx="0.000153302092922362"
@@ -106,5 +112,5 @@
         rpy="0 0 0" />
       <mass
-        value="0.18653997068198" />
+        value="${wheel_mass}" />
       <inertia
         ixx="0.000153302490492137"
@@ -159,5 +165,5 @@
         rpy="0 0 0" />
       <mass
-        value="0.186539970674412" />
+        value="${wheel_mass}" />
       <inertia
         ixx="0.000153302490497661"
@@ -212,5 +218,5 @@
         rpy="0 0 0" />
       <mass
-        value="0.186539971470881" />
+        value="${wheel_mass}" />
       <inertia
         ixx="0.000153302490504048"
@@ -265,5 +271,5 @@
         rpy="0 0 0" />
       <mass
-        value="3.83878903165985" />
+        value="${lidar_mass}" />
       <inertia
         ixx="0.0179107890685936"
@@ -320,5 +326,5 @@
         rpy="0 0 0" />
       <mass
-        value="0.658408070652594" />
+        value="${kinect_mass}" />
       <inertia
         ixx="0.000269628323265001"

Commit message: add tansmission

File: kinetic/src/four_wheel_urdf/urdf/four_wheel_urdf.urdf.xacro (robot description, xacro)
@@ -5,7 +5,34 @@
      For more information, please see http://wiki.ros.org/sw_urdf_exporter -->
 <!--Model constructed by yu zhuotong 2020.5.10-->
+<!--mass property-->
   <xacro:property name = "wheel_mass" value = "0.5"/>
   <xacro:property name = "lidar_mass" value = "2"/>
   <xacro:property name = "kinect_mass" value = "0.5"/>
+<!--simplified wheel collision model-->
+  <xacro:macro name = "wheel_shape">
+    <cylinder radius="${0.14/2}" length="0.01"/>
+  </xacro:macro>
+<!--add physical properties and transmissions for wheels-->
+  <xacro:macro name = "wheel_property" params="prefix suffix">
+  <!--physical properties for gazebo simulator-->
+    <gazebo reference="${prefix}_${suffix}_wheel">
+      <mu1 value="200.0"/>
+      <mu2 value="100.0"/>
+      <kp value="10000000.0" />
+      <kd value="1.0" />
+      <material>Gazebo/Grey</material>
+    </gazebo>
+  <!--transmissions-->
+    <transmission name="${prefix}_${suffix}_wheel_trans">
+      <type>transmission_interface/SimpleTransmission</type>
+      <actuator name="${prefix}_${suffix}_motor">
+        <mechanicalReduction>1</mechanicalReduction>
+      </actuator>
+      <joint name="${prefix}_${suffix}_joint">
+        <hardwareInterface>VelocityJointInterface</hardwareInterface>
+      </joint>
+    </transmission>
+  </xacro:macro>
+  <!--the main part begins here                                             -->
   <link
     name="base_link">
@@ -264,4 +291,8 @@
       xyz="0 0 1" />
   </joint>
+<xacro:wheel_property prefix = "back" suffix ="left"/>
+<xacro:wheel_property prefix = "back" suffix ="right"/>
+<xacro:wheel_property prefix = "front" suffix ="left"/>
+<xacro:wheel_property prefix = "front" suffix ="right"/>
   <link
     name="lidar_link">

Commit message: simplified collision

File: kinetic/src/four_wheel_urdf/urdf/four_wheel_urdf.urdf.xacro (robot description, xacro)
@@ -11,5 +11,5 @@
 <!--simplified wheel collision model-->
   <xacro:macro name = "wheel_shape">
-    <cylinder radius="${0.14/2}" length="0.01"/>
+    <cylinder radius="${0.10/2}" length="0.06"/>
   </xacro:macro>
 <!--add physical properties and transmissions for wheels-->
@@ -34,5 +34,5 @@
     </transmission>
   </xacro:macro>
-  <!--the main part begins here                                             -->
+  <!--the main part begins here -->
   <link
     name="base_link">
@@ -114,6 +114,9 @@
         rpy="0 0 0" />
       <geometry>
+      <xacro:wheel_shape/>
+       <!--
         <mesh
           filename="package://four_wheel_urdf/meshes/front_left_wheel.STL" />
+          -->
       </geometry>
     </collision>
@@ -167,6 +170,9 @@
         rpy="0 0 0" />
       <geometry>
+        <xacro:wheel_shape/>
+       <!--
         <mesh
           filename="package://four_wheel_urdf/meshes/front_right_wheel.STL" />
+          -->
       </geometry>
     </collision>
@@ -220,6 +226,9 @@
         rpy="0 0 0" />
       <geometry>
+      <xacro:wheel_shape/>
+       <!--
         <mesh
           filename="package://four_wheel_urdf/meshes/back_left_wheel.STL" />
+          -->
       </geometry>
     </collision>
@@ -273,6 +282,9 @@
         rpy="0 0 0" />
       <geometry>
+      <xacro:wheel_shape/>
+       <!--
         <mesh
           filename="package://four_wheel_urdf/meshes/back_right_wheel.STL" />
+          -->
       </geometry>
     </collision>

Commit message: correct diff_drive

File: kinetic/src/four_wheel_urdf/urdf/four_wheel_urdf.urdf.xacro (robot description, xacro)
@@ -6,10 +6,10 @@
 <!--Model constructed by yu zhuotong 2020.5.10-->
 <!--mass property-->
-  <xacro:property name = "wheel_mass" value = "0.5"/>
+  <xacro:property name = "wheel_mass" value = "0.6"/>
   <xacro:property name = "lidar_mass" value = "2"/>
-  <xacro:property name = "kinect_mass" value = "0.5"/>
+  <xacro:property name = "kinect_mass" value = "0.4"/>
 <!--simplified wheel collision model-->
   <xacro:macro name = "wheel_shape">
-    <cylinder radius="${0.10/2}" length="0.06"/>
+    <cylinder radius="${0.10/2}" length="0.005"/>
   </xacro:macro>
 <!--add physical properties and transmissions for wheels-->
@@ -42,5 +42,5 @@
         rpy="0 0 0" />
       <mass
-        value="2.37412974413616" />
+        value="3.37412974413616" />
       <inertia
         ixx="0.0108285754206111"
@@ -126,6 +126,6 @@
     type="continuous">
     <origin
-      xyz="0.137625631329235 0.15756248166201 -0.0123743686707646"
-      rpy="1.5707963267949 -1.09222488301814 0" />
+      xyz="0.137625631329235 0.19056248166201 -0.0123743686707646"
+      rpy="1.5707963267949 0 3.14159265358979" /> <!--original: 0.15756248166201-->
     <parent
       link="base_link" />
@@ -182,6 +182,6 @@
     type="continuous">
     <origin
-      xyz="0.137625631329235 -0.15756248166201 -0.0123743686707646"
-      rpy="-1.57079632679489 -1.54165987688924 3.14159265358979" />
+      xyz="0.137625631329235 -0.19056248166201 -0.0123743686707646"
+      rpy="1.5707963267949 0 3.14159265358979" />
     <parent
       link="base_link" />
@@ -238,6 +238,6 @@
     type="continuous">
     <origin
-      xyz="-0.137625631329235 0.15756248166201 -0.0123743686707646"
-      rpy="1.5707963267949 0.972888437481976 0" />
+      xyz="-0.137625631329235 0.19056248166201 -0.0123743686707646"
+      rpy="1.5707963267949 0 3.14159265358979" />
     <parent
       link="base_link" />
@@ -294,6 +294,6 @@
     type="continuous">
     <origin
-      xyz="-0.137625631329235 -0.15756248166201 -0.0123743686707645"
-      rpy="1.5707963267949 -1.50975652463866 0" />
+      xyz="-0.137625631329235 -0.19056248166201 -0.0123743686707645"
+      rpy="1.5707963267949 0 3.14159265358979" />
     <parent
       link="base_link" />

Commit message: add gmapping based on lidar

File: kinetic/src/four_wheel_urdf/urdf/four_wheel_urdf.urdf.xacro (robot description, xacro)
@@ -325,9 +325,9 @@
     <visual>
       <origin
-        xyz="0 0 0"
-        rpy="0 0 0" />
-      <geometry>
-        <mesh
-          filename="package://four_wheel_urdf/meshes/lidar_link.STL" />
+        xyz="-0.17 0 0"
+        rpy="0 0 0" />
+      <geometry>
+        <mesh
+          filename="package://four_wheel_urdf/meshes/hokuyo.dae" />
       </geometry>
       <material
@@ -353,6 +353,6 @@
     type="fixed">
     <origin
-      xyz="0.10636719253573 0 0.084"
-      rpy="1.5707963267949 0 1.5707963267949" />
+      xyz="0.34236719253573 0 0.118"
+      rpy="0 0 0" />
     <parent
       link="base_link" />
@@ -362,4 +362,40 @@
       xyz="0 0 0" />
   </joint>
+ <!-- hokuyo -->
+  <gazebo reference="lidar_link">
+    <sensor type="ray" name="head_hokuyo_sensor">
+      <pose>0 0 0 0 0 0</pose>
+      <visualize>false</visualize>
+      <update_rate>40</update_rate>
+      <ray>
+        <scan>
+          <horizontal>
+            <samples>720</samples>
+            <resolution>1</resolution>
+            <min_angle>-2.35619</min_angle>
+            <max_angle>2.35619</max_angle>
+          </horizontal>
+        </scan>
+        <range>
+          <min>0.10</min>
+          <max>30</max>
+          <resolution>0.01</resolution>
+        </range>
+        <noise>
+          <type>gaussian</type>
+          <!-- Noise parameters based on published spec for Hokuyo laser
+               achieving "+-30mm" accuracy at range < 10m.  A mean of 0.0m and
+               stddev of 0.01m will put 99.7% of samples within 0.03m of the true
+               reading. -->
+          <mean>0.0</mean>
+          <stddev>0.01</stddev>
+        </noise>
+      </ray>
+      <plugin name="gazebo_ros_head_hokuyo_controller" filename="libgazebo_ros_laser.so">
+        <topicName>scan</topicName>
+        <frameName>lidar_link</frameName>
+      </plugin>
+    </sensor>
+  </gazebo>
   <link
     name="kinect_link">

Commit message: Hokuyo lidar

File: kinetic/src/four_wheel_urdf/urdf/four_wheel_urdf.urdf.xacro (robot description, xacro)
@@ -7,5 +7,5 @@
 <!--mass property-->
   <xacro:property name = "wheel_mass" value = "0.6"/>
-  <xacro:property name = "lidar_mass" value = "2"/>
+  <xacro:property name = "lidar_mass" value = "0.8"/>
   <xacro:property name = "kinect_mass" value = "0.4"/>
 <!--simplified wheel collision model-->
@@ -444,5 +444,5 @@
     type="fixed">
     <origin
-      xyz="0.15 0 0.31"
+      xyz="0.15 0 0.22"
       rpy="3.14159265358979 0 1.5707963267949" />
     <parent
@@ -460,5 +460,5 @@
         rpy="0 0 0" />
       <mass
-        value="0.176384011821692" />
+        value="1.176384011821692" />
       <inertia
         ixx="6.51045221494184E-05"
@@ -515,5 +515,5 @@
         rpy="0 0 0" />
       <mass
-        value="0.0275146541367252" />
+        value="0.5275146541367252" />
       <inertia
         ixx="3.2123731049697E-06"

Commit message: Change Appearance

File: kinetic/src/four_wheel_urdf/urdf/four_wheel_urdf.urdf.xacro (robot description, xacro)
@@ -416,9 +416,9 @@
     <visual>
       <origin
-        xyz="0 0 0"
-        rpy="3.14159265 0 1.570796325" />
-      <geometry>
-        <mesh
-          filename="package://four_wheel_urdf/meshes/kinect_link.STL" />
+        xyz="0 0 0.0218"
+        rpy="0 0 1.570796325" />
+      <geometry>
+        <mesh
+          filename="package://four_wheel_urdf/meshes/kinect.dae" />
       </geometry>
       <material
@@ -538,4 +538,7 @@
     -->
   </link>
+  <gazebo reference="raspberry_link">
+      <material>Gazebo/Grey</material>
+  </gazebo>
   <joint
     name="raspberry_joint"
@@ -593,4 +596,7 @@
     -->
   </link>
+  <gazebo reference="driver_link">
+      <material>Gazebo/Grey</material>
+  </gazebo>
   <joint
     name="driver_joint"

File: kinetic/src/four_wheel_urdf/urdf/two_wheel_urdf.urdf.xacro (robot description, xacro)
@@ -432,9 +432,9 @@
     <visual>
       <origin
-        xyz="0 0 0"
-        rpy="3.14159265 0 1.570796325" />
-      <geometry>
-        <mesh
-          filename="package://four_wheel_urdf/meshes/kinect_link.STL" />
+        xyz="0 0 0.0218"
+        rpy="0 0 1.570796325" />
+      <geometry>
+        <mesh
+          filename="package://four_wheel_urdf/meshes/kinect.dae" />
       </geometry>
       <material
@@ -554,4 +554,7 @@
     -->
   </link>
+  <gazebo reference="raspberry_link">
+      <material>Gazebo/Grey</material>
+  </gazebo>
   <joint
     name="raspberry_joint"
@@ -609,4 +612,7 @@
     -->
   </link>
+  <gazebo reference="driver_link">
+      <material>Gazebo/Grey</material>
+  </gazebo>
   <joint
     name="driver_joint"
